Commit message: can execute

File: config/robot.urdf.xacro (robot description, xacro)
@@ -9,8 +9,8 @@
     <origin xyz="0 0 0" rpy="0 0 0" />
   </joint>
-  <link name="lidar_link"> </link>
+  <link name="hesai_lidar"> </link>
   <joint name="lidar_joint" type="fixed">
     <parent link="base_link" />
-    <child link="lidar_link" />
+    <child link="hesai_lidar" />
     <origin xyz="0 0 0" rpy="0 0 0" />
   </joint>
